Commit message: mike

File: ur5_with_asus_description/urdf/ur5_with_asus_joint_limited_robot.urdf.xacro (robot description, xacro)
@@ -8,5 +8,5 @@
   <xacro:include filename="$(find hector_sensors_description)/urdf/asus_camera.urdf.xacro"/>
   <xacro:asus_camera name="camera" parent="ee_link">
-     <origin xyz="-0.0376392422473 -0.0893148572862 0.0678378626701" rpy=" 0.77814092516 -0.0349196137731 0.0446712637898"/>
+    <origin xyz="-0.0374273994792 -0.0595613873455 0.0735889802814" rpy="0.752115280096 -0.169022608744 -0.21601697481"/>
   </xacro:asus_camera>
   <!-- arm -->
@@ -17,4 +17,5 @@
     <child link="base_link"/>
     <origin xyz="0.0 0.0 0.98" rpy="0.0 0.0 0.0"/>
+    <!--<origin xyz="0.0 0.0 0." rpy="0.0 0.0 0.0"/>-->
   </joint>
 </robot>
